Commit message: mecanum control

File: turtlebot3_description/urdf/turtlebot3_mecanum.urdf.xacro (robot description, xacro)
@@ -1,4 +1,4 @@
 <?xml version="1.0" ?>
-<robot name="turtlebot3_mecanum" xmlns:xacro="http://ros.org/wiki/xacro">
+<robot name="turtlebot3_waffle_pi_for_open_manipulator" xmlns:xacro="http://ros.org/wiki/xacro">
   <xacro:include filename="$(find turtlebot3_description)/urdf/common_properties.xacro"/>
   <xacro:include filename="$(find turtlebot3_description)/urdf/turtlebot3_waffle_pi_for_open_manipulator.gazebo.xacro"/>
@@ -34,61 +34,5 @@
     </inertial>
   </link>
-  <joint name="r_wheel_left_joint" type="continuous">
-    <parent link="base_link"/>
-    <child link="r_wheel_left_link"/>
-    <origin xyz="-0.144 0.144 0.023" rpy="-1.57 0 0"/>
-    <axis xyz="0 0 1"/>
-  </joint>
-  <link name="r_wheel_left_link">
-    <visual>
-      <origin xyz="0 0 0" rpy="1.57 0 0"/>
-      <geometry>
-        <mesh filename="package://turtlebot3_description/meshes/wheels/left_tire.stl" scale="0.001 0.001 0.001"/>
-      </geometry>
-      <material name="dark"/>
-    </visual>
-    <collision>
-      <origin xyz="0 0 0" rpy="0 0 0"/>
-      <geometry>
-        <cylinder length="0.018" radius="0.033"/>
-      </geometry>
-    </collision>
-    <inertial>
-      <origin xyz="0 0 0" />
-      <mass value="2.8498940e-02" />
-      <inertia ixx="1.1175580e-05" ixy="-4.2369783e-11" ixz="-5.9381719e-09"
-               iyy="1.1192413e-05" iyz="-1.4400107e-11"
-               izz="2.0712558e-05" />
-      </inertial>
-  </link>
-  <joint name="r_wheel_right_joint" type="continuous">
-    <parent link="base_link"/>
-    <child link="r_wheel_right_link"/>
-    <origin xyz="-0.144 -0.144 0.023" rpy="-1.57 0 0"/>
-    <axis xyz="0 0 1"/>
-  </joint>
-  <link name="r_wheel_right_link">
-    <visual>
-      <origin xyz="0 0 0" rpy="1.57 0 0"/>
-      <geometry>
-        <mesh filename="package://turtlebot3_description/meshes/wheels/right_tire.stl" scale="0.001 0.001 0.001"/>
-      </geometry>
-      <material name="dark"/>
-    </visual>
-    <collision>
-      <origin xyz="0 0.001 0" rpy="0 0 0"/>
-      <geometry>
-        <cylinder length="0.018" radius="0.033"/>
-      </geometry>
-    </collision>
-    <inertial>
-      <origin xyz="0 0 0" />
-      <mass value="2.8498940e-02" />
-      <inertia ixx="1.1175580e-05" ixy="-4.2369783e-11" ixz="-5.9381719e-09"
-               iyy="1.1192413e-05" iyz="-1.4400107e-11"
-               izz="2.0712558e-05" />
-      </inertial>
-  </link>
-  <joint name="wheel_left_joint" type="continuous">
+  <joint name="wheel_left_front_joint" type="continuous">
     <parent link="base_link"/>
     <child link="wheel_left_link"/>
@@ -118,5 +62,5 @@
       </inertial>
   </link>
-  <joint name="wheel_right_joint" type="continuous">
+  <joint name="wheel_right_front_joint" type="continuous">
     <parent link="base_link"/>
     <child link="wheel_right_link"/>
@@ -125,4 +69,60 @@
   </joint>
   <link name="wheel_right_link">
+    <visual>
+      <origin xyz="0 0 0" rpy="1.57 0 0"/>
+      <geometry>
+        <mesh filename="package://turtlebot3_description/meshes/wheels/right_tire.stl" scale="0.001 0.001 0.001"/>
+      </geometry>
+      <material name="dark"/>
+    </visual>
+    <collision>
+      <origin xyz="0 0.001 0" rpy="0 0 0"/>
+      <geometry>
+        <cylinder length="0.018" radius="0.033"/>
+      </geometry>
+    </collision>
+    <inertial>
+      <origin xyz="0 0 0" />
+      <mass value="2.8498940e-02" />
+      <inertia ixx="1.1175580e-05" ixy="-4.2369783e-11" ixz="-5.9381719e-09"
+               iyy="1.1192413e-05" iyz="-1.4400107e-11"
+               izz="2.0712558e-05" />
+      </inertial>
+  </link>
+  <joint name="wheel_left_rear_joint" type="continuous">
+    <parent link="base_link"/>
+    <child link="wheel_left_rear_link"/>
+    <origin xyz="-0.15 0.144 0.023" rpy="-1.57 0 0"/>
+    <axis xyz="0 0 1"/>
+  </joint>
+  <link name="wheel_left_rear_link">
+    <visual>
+      <origin xyz="0 0 0" rpy="1.57 0 0"/>
+      <geometry>
+        <mesh filename="package://turtlebot3_description/meshes/wheels/left_tire.stl" scale="0.001 0.001 0.001"/>
+      </geometry>
+      <material name="dark"/>
+    </visual>
+    <collision>
+      <origin xyz="0 0 0" rpy="0 0 0"/>
+      <geometry>
+        <cylinder length="0.018" radius="0.033"/>
+      </geometry>
+    </collision>
+    <inertial>
+      <origin xyz="0 0 0" />
+      <mass value="2.8498940e-02" />
+      <inertia ixx="1.1175580e-05" ixy="-4.2369783e-11" ixz="-5.9381719e-09"
+               iyy="1.1192413e-05" iyz="-1.4400107e-11"
+               izz="2.0712558e-05" />
+      </inertial>
+  </link>
+  <joint name="wheel_right_rear_joint" type="continuous">
+    <parent link="base_link"/>
+    <child link="wheel_right_rear_link"/>
+    <origin xyz="-0.15 -0.144 0.023" rpy="-1.57 0 0"/>
+    <axis xyz="0 0 1"/>
+  </joint>
+  <link name="wheel_right_rear_link">
     <visual>
       <origin xyz="0 0 0" rpy="1.57 0 0"/>

Commit message: add mecanum urdf & teleop

File: turtlebot3_description/urdf/turtlebot3_mecanum.urdf.xacro (robot description, xacro)
@@ -34,5 +34,5 @@
     </inertial>
   </link>
-  <joint name="wheel_left_front_joint" type="continuous">
+  <joint name="wheel_left_joint" type="continuous">
     <parent link="base_link"/>
     <child link="wheel_left_link"/>
@@ -62,5 +62,5 @@
       </inertial>
   </link>
-  <joint name="wheel_right_front_joint" type="continuous">
+  <joint name="wheel_right_joint" type="continuous">
     <parent link="base_link"/>
     <child link="wheel_right_link"/>
@@ -90,11 +90,11 @@
       </inertial>
   </link>
-  <joint name="wheel_left_rear_joint" type="continuous">
-    <parent link="base_link"/>
-    <child link="wheel_left_rear_link"/>
+  <joint name="wheel_r_left_joint" type="continuous">
+    <parent link="base_link"/>
+    <child link="wheel_r_left_link"/>
     <origin xyz="-0.15 0.144 0.023" rpy="-1.57 0 0"/>
     <axis xyz="0 0 1"/>
   </joint>
-  <link name="wheel_left_rear_link">
+  <link name="wheel_r_left_link">
     <visual>
       <origin xyz="0 0 0" rpy="1.57 0 0"/>
@@ -118,11 +118,11 @@
       </inertial>
   </link>
-  <joint name="wheel_right_rear_joint" type="continuous">
-    <parent link="base_link"/>
-    <child link="wheel_right_rear_link"/>
+  <joint name="wheel_r_right_joint" type="continuous">
+    <parent link="base_link"/>
+    <child link="wheel_r_right_link"/>
     <origin xyz="-0.15 -0.144 0.023" rpy="-1.57 0 0"/>
     <axis xyz="0 0 1"/>
   </joint>
-  <link name="wheel_right_rear_link">
+  <link name="wheel_r_right_link">
     <visual>
       <origin xyz="0 0 0" rpy="1.57 0 0"/>
